Commit message: Correcciones de computadora LABME, correccion de cambio de unidades y archivo .xacro

File: cobot_description/urdf/Largo/cobot.urdf.xacro (robot description, xacro)
@@ -34,10 +34,10 @@
     <xacro:property name="limit_low_elbow_rotation" value="-2.793" />
     <xacro:property name="limit_up_elbow_rotation" value="2.793" />
-    <xacro:property name="limit_low_forearm_rotation" value="-3.05433" />    <!-- original -3.05433  -->
-    <xacro:property name="limit_up_forearm_rotation" value="3.05433" />      <!-- original 3.05433  -->
-    <xacro:property name="limit_low_wrist_rotation" value="-3.05433" />
-    <xacro:property name="limit_up_wrist_rotation" value="3.05433" />
-    <xacro:property name="limit_low_hand_rotation" value="-3.05433" />
-    <xacro:property name="limit_up_hand_rotation" value="3.05433" />
+    <xacro:property name="limit_low_forearm_rotation" value="-2.5307274125" />    <!-- 150 grados -->
+    <xacro:property name="limit_up_forearm_rotation" value="2.5307274125" />
+    <xacro:property name="limit_low_wrist_rotation" value="-2.5307274125" />
+    <xacro:property name="limit_up_wrist_rotation" value="2.5307274125" />
+    <xacro:property name="limit_low_hand_rotation" value="-2.5307274125" />
+    <xacro:property name="limit_up_hand_rotation" value="2.5307274125" />
 	<!-- Links -->
     <link name="world"/>

File: cobot_description/urdf/corto girado/cobot.urdf.xacro (robot description, xacro)
@@ -172,5 +172,5 @@
         <parent link="elbow_link" />
         <child link="forearm_link" />
-        <origin xyz="-0.00050 -0.04300 0.17050" rpy="0 0 0" />
+        <origin xyz="-0.00050 -0.01300 0.17050" rpy="0 0 0" />
 		<limit effort="1" velocity="1.0" lower="${limit_low_forearm_rotation}" upper="${limit_up_forearm_rotation}" />
 		<axis xyz="0 1 0" />
@@ -186,5 +186,5 @@
         <parent link="wrist_link" />
         <child link="hand_link" />
-        <origin xyz=" 0.00053 -0.01470 0.05875 " rpy="0 0 0" />
+        <origin xyz=" -0.00053 0.01470 0.05875 " rpy="0 0 0" />
 		<limit effort="1" velocity="1.0" lower="${limit_low_hand_rotation}" upper="${limit_up_hand_rotation}" />
 		<axis xyz="0 1 0" />
