Commit message: Correcciones de ejecucion de trayectorias

File: cobot_description/urdf/cobot.urdf.xacro (robot description, xacro)
@@ -167,5 +167,5 @@
         <origin xyz="-0.00035 0.00735 0.22543" rpy="0 0 0" />
 		<limit effort="1" velocity="1.0" lower="${limit_low_elbow_rotation}" upper="${limit_up_elbow_rotation}" />
-		<axis xyz="0 1 0" />
+		<axis xyz="0 -1 0" />
 	</joint>
 	<joint name="joint_4" type="revolute">

Commit message: Correcciones varias

File: cobot_description/urdf/cobot.urdf.xacro (robot description, xacro)
@@ -30,14 +30,14 @@
     <xacro:property name="limit_low_shoulder_rotation" value="-3.05433" />
     <xacro:property name="limit_up_shoulder_rotation" value="3.05433" />
-    <xacro:property name="limit_low_arm_rotation" value="-1.91986" />
-    <xacro:property name="limit_up_arm_rotation" value="0.640187" />
-    <xacro:property name="limit_low_elbow_rotation" value="-1.397485" />
-    <xacro:property name="limit_up_elbow_rotation" value="${PI/2}" />
-    <xacro:property name="limit_low_forearm_rotation" value="-1.58" />    <!-- original -3.05433  -->
-    <xacro:property name="limit_up_forearm_rotation" value="1.58" />      <!-- original 3.05433  -->
-    <xacro:property name="limit_low_wrist_rotation" value="-1.74533" />
-    <xacro:property name="limit_up_wrist_rotation" value="1.91986" />
-    <xacro:property name="limit_low_hand_rotation" value="-2.57436" />
-    <xacro:property name="limit_up_hand_rotation" value="2.57436" />
+    <xacro:property name="limit_low_arm_rotation" value="-2.0072" />
+    <xacro:property name="limit_up_arm_rotation" value="2.0072" />
+    <xacro:property name="limit_low_elbow_rotation" value="-2.793" />
+    <xacro:property name="limit_up_elbow_rotation" value="2.793" />
+    <xacro:property name="limit_low_forearm_rotation" value="-3.05433" />    <!-- original -3.05433  -->
+    <xacro:property name="limit_up_forearm_rotation" value="3.05433" />      <!-- original 3.05433  -->
+    <xacro:property name="limit_low_wrist_rotation" value="-3.05433" />
+    <xacro:property name="limit_up_wrist_rotation" value="3.05433" />
+    <xacro:property name="limit_low_hand_rotation" value="-3.05433" />
+    <xacro:property name="limit_up_hand_rotation" value="3.05433" />
 	<!-- Links -->
     <link name="world"/>

Commit message: Cambio de xacro y diseño a robot petacon

File: cobot_description/urdf/cobot.urdf.xacro (robot description, xacro)
@@ -165,5 +165,5 @@
         <parent link="arm_link" />
         <child link="elbow_link" />
-        <origin xyz="-0.00035 0.00735 0.22543" rpy="0 0 0" />
+        <origin xyz="-0.00005 0.00735 0.17466" rpy="0 0 0" />
 		<limit effort="1" velocity="1.0" lower="${limit_low_elbow_rotation}" upper="${limit_up_elbow_rotation}" />
 		<axis xyz="0 -1 0" />
@@ -172,5 +172,5 @@
         <parent link="elbow_link" />
         <child link="forearm_link" />
-        <origin xyz="0.00010 -0.01300 0.22127" rpy="0 0 0" />
+        <origin xyz="-0.00050 -0.01300 0.17050" rpy="0 0 0" />
 		<limit effort="1" velocity="1.0" lower="${limit_low_forearm_rotation}" upper="${limit_up_forearm_rotation}" />
 		<axis xyz="0 1 0" />

Commit message: correccion .xacro3

File: cobot_description/urdf/cobot.urdf.xacro (robot description, xacro)
@@ -179,5 +179,5 @@
         <parent link="forearm_link" />
         <child link="wrist_link" />
-		<origin xyz=" -0.00083 0.05875 0.01530 " rpy="0 0 0" />
+		<origin xyz=" 0.00083 -0.05875 0.01530 " rpy="0 0 0" />
 		<limit effort="1" velocity="1.0" lower="${limit_low_wrist_rotation}" upper="${limit_up_wrist_rotation}" />
 		<axis xyz="0 0 1" />
@@ -186,5 +186,5 @@
         <parent link="wrist_link" />
         <child link="hand_link" />
-        <origin xyz=" 0.00053 -0.01470 0.05875 " rpy="0 0 0" />
+        <origin xyz=" 0.00053 -0.01470 0.05875 " rpy="0 0 135" />
 		<limit effort="1" velocity="1.0" lower="${limit_low_hand_rotation}" upper="${limit_up_hand_rotation}" />
 		<axis xyz="0 1 0" />

Commit message: Correcciones .xacro4

File: cobot_description/urdf/cobot.urdf.xacro (robot description, xacro)
@@ -186,5 +186,5 @@
         <parent link="wrist_link" />
         <child link="hand_link" />
-        <origin xyz=" 0.00053 -0.01470 0.05875 " rpy="0 0 135" />
+        <origin xyz=" 0.00053 -0.01470 0.05875 " rpy="0 0 0" />
 		<limit effort="1" velocity="1.0" lower="${limit_low_hand_rotation}" upper="${limit_up_hand_rotation}" />
 		<axis xyz="0 1 0" />
@@ -193,5 +193,5 @@
         <parent link="hand_link" />
         <child link="tool_link" />
-        <origin xyz="0 0.04 0" rpy="0 0 0" />
+        <origin xyz="0 -0.04 0" rpy="0 0 0" />
 	</joint>
 </robot>
